File: kicad/ember.kicad_pcb (KiCad board)
At the start: 2 copper layers, 75 x 52.5 mm, 16 parts, among them J1 Battery 6xAA, J2 Igniter, Q1 IRF3205, Q2 BC547, SW1 Arm Switch, SW2 Push Button

Commit message: added launch controller models
Parts:
- added M3: MountingHole_3.2mm_M3, MountingHole:MountingHole_3.2mm_M3, F.Cu at (117.6, 102.4)
- added M3: MountingHole_3.2mm_M3, MountingHole:MountingHole_3.2mm_M3, F.Cu at (169.3, 106.1)
- added M3: MountingHole_3.2mm_M3, MountingHole:MountingHole_3.2mm_M3, F.Cu at (146.3, 102.4)
