File: kicad/ember_flight_recorder/ember_flight_recorder.kicad_pcb (KiCad board)
At the start: 2 copper layers, 0 parts

Commit message: updated footprint and 3d models
Parts:
- added BT1: LiPo battery, Connector_Wire:SolderWire-0.75sqmm_1x02_P7mm_D1.25mm_OD3.5mm, F.Cu at (153.6, 115.6)
- added C1: 0.1uF, Capacitor_SMD:C_1206_3216Metric_Pad1.33x1.80mm_HandSolder, F.Cu at (174.1, 110.7)
- added C2: 100uF, Capacitor_SMD:C_1206_3216Metric_Pad1.33x1.80mm_HandSolder, F.Cu at (174.1, 114.0)
- added C3: 1uF, Capacitor_SMD:C_1206_3216Metric_Pad1.33x1.80mm_HandSolder, F.Cu at (174.1, 117.4)
- added C4: 1uF, Capacitor_SMD:C_1206_3216Metric_Pad1.33x1.80mm_HandSolder, F.Cu at (174.1, 120.7)
- added C5: 10uF, Capacitor_SMD:C_1206_3216Metric_Pad1.33x1.80mm_HandSolder, F.Cu at (174.1, 124.1)
- added C6: 100nF, Capacitor_SMD:C_1206_3216Metric_Pad1.33x1.80mm_HandSolder, F.Cu at (174.1, 127.4)
- added D5: LED, LED_SMD:LED_1210_3225Metric_Pad1.42x2.65mm_HandSolder, F.Cu at (163.3, 125.7)
- added Q3: FS8205A, FS8205A:SOT-23-6L_TCP-M, F.Cu at (163.4, 121.0)
- added Q4: AO3401A, Package_TO_SOT_SMD:SOT-23, F.Cu at (153.1, 120.6)
- added R5: 330, Resistor_SMD:R_0805_2012Metric_Pad1.20x1.40mm_HandSolder, F.Cu at (157.9, 119.9)
- added R6: 2.2k, Resistor_SMD:R_0805_2012Metric_Pad1.20x1.40mm_HandSolder, F.Cu at (157.9, 122.8)
- added R7: 100, Resistor_SMD:R_0805_2012Metric_Pad1.20x1.40mm_HandSolder, F.Cu at (157.9, 125.8)
- added U2: DW01A, Package_TO_SOT_SMD:SOT-23-6, F.Cu at (166.2, 115.2)
- added U3: MCP1700x-330xxTT, Package_TO_SOT_SMD:SOT-23, F.Cu at (153.1, 125.1)
- added U4: module_mpu6050, usini_sensors:module_mpu6050, F.Cu at (173.0, 107.2)
- added U5: module_bme280, usini_sensors:module_bme280, F.Cu at (183.8, 123.3)
- added U6: ESP32-C3_SUPERMINI_SMD, smd:MODULE_ESP32-C3_SUPERMINI, F.Cu at (160.9, 100.7)
