File: kicad/ember_flight_recorder/ember_flight_recorder.kicad_pcb (KiCad board)
At the start: 2 copper layers, 18 parts, among them Q3 FS8205A, Q4 AO3401A, U2 DW01A, U3 MCP1700x-330xxTT, U4 module_mpu6050, U5 module_bme280, U6 ESP32-C3_SUPERMINI_SMD

Commit message: flight recorder rev1
Parts:
- added SW1: SW_SPDT, Button_Switch_THT:SW_Slide-03_Wuerth-WS-SLTV_10x2.5x6.4_P2.54mm, F.Cu at (145.8, 120.2)
- C2, C3, C4, C5, C6, D5, R7, U4: moved to B.Cu
- moved U5 52.2 mm to (148.7, 84.6), turned to 180 degrees
- moved C6 49.7 mm to (142.3, 89.2), turned to 90 degrees
- moved U4 48.7 mm to (131.5, 81.6)
- moved C4 39.6 mm to (136.2, 109.5), turned to -90 degrees
- moved C5 38.3 mm to (138.7, 109.5), turned to -90 degrees
- moved D5 37.8 mm to (141.8, 94.6), turned to 180 degrees
- moved R7 29.8 mm to (144.4, 99.2), turned to -90 degrees
- moved C3 27.8 mm to (146.8, 112.4), turned to 90 degrees
- moved C1 24.5 mm to (149.7, 109.8), turned to -90 degrees
- moved C2 24.1 mm to (150.1, 112.3), turned to 90 degrees
- moved Q3 21.8 mm to (142.5, 114.9)
- moved U3 21.7 mm to (135.0, 113.1), turned to -90 degrees
- moved U6 20.2 mm to (142.7, 91.8)
- moved BT1 18.0 mm to (139.2, 126.5)
- moved U2 17.7 mm to (148.6, 114.9)
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Connections:
- BT1 pad 2: GND -> GNDPWR
- C1 pad 2: GND -> Net-(SW1-C)
- Q3 pad 1: GND -> Net-(SW1-C)
- Q4 pad 1: GND -> GNDPWR
- U2 pad 6: GND -> Net-(SW1-C)
- U6 pad 1: Net-(D5-A) -> unconnected-(U6-GPIO1-Pad1)
- U6 pad 10: unconnected-(U6-GPIO10-Pad10) -> Net-(D5-A)
Routing:
- net GND: track 0.00 -> 115.8 mm, vias 0 -> 6
- net VOUT_3V3: track 0.00 -> 64.3 mm, vias 0 -> 3
- net Net-(U4-SDA): track 0.00 -> 37.0 mm, vias 0 -> 1
- net Net-(U4-SCL): track 0.00 -> 32.8 mm, vias 0 -> 1
- net Net-(Q4-S): track 0.00 -> 27.7 mm, vias 0 -> 2
- net Net-(SW1-C): track 0.00 -> 19.6 mm
- net GNDPWR: track 0.00 -> 19.5 mm
- net Net-(U2-VCC): track 0.00 -> 13.3 mm
- net Net-(U2-CS): track 0.00 -> 10.9 mm
- net Net-(BT1-+): track 0.00 -> 6.95 mm
- net Net-(D5-A): track 0.00 -> 5.60 mm, vias 0 -> 1
- net Net-(D5-K): track 0.00 -> 4.06 mm
- net Net-(U2-OD): track 0.00 -> 3.52 mm
- net Net-(U2-OC): track 0.00 -> 3.52 mm
- added copper zone on B.Cu, net GND
- added copper zone on F.Cu, net GND
- added copper zone on B.Cu, net VOUT_3V3
- added copper zone on F.Cu, net VOUT_3V3
Other:
- board outline added: 25 x 50 mm

Commit message: flight recorder rev2
Routing:
- net Net-(U4-SCL): track 32.8 -> 36.6 mm
- net Net-(U4-SDA): track 37.0 -> 33.3 mm
- net VOUT_3V3: track 64.3 -> 66.9 mm
Other:
- board text added: "*"
