File: kicad/ember_launch_controller/ember_launch_controller.kicad_pcb (KiCad board)
At the start: 2 copper layers, 75 x 52.5 mm, 19 parts, among them J1 Battery 6xAA, J2 Igniter, M3 MountingHole_3.2mm_M3, Q1 IRF3205, Q2 BC547, SW1 Arm Switch, SW2 Push Button

Commit message: restructured kicad project
Parts:
- D2: value Green LED -> Green
- D3: value Red LED -> Red
- D4: value Blue LED -> Blue
- Q2: footprint Package_TO_SOT_THT:TO-92L_HandSolder -> Package_TO_SOT_THT:TO-92_Inline

Commit message: more gerber files
Parts:
- Q2: footprint Package_TO_SOT_THT:TO-92_Inline -> Package_TO_SOT_THT:TO-92L_HandSolder
Routing:
- net GND: track 182.4 -> 183.2 mm
- removed copper zone on B.Cu, net (none)
- removed copper zone on F.Cu, net (none)
Changed lines of the file:
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@@
 			(outputformat 1)
 			(mirror no)
-			(drillshape 1)
+			(drillshape 0)
 			(scaleselection 1)
-			(outputdirectory "")
+			(outputdirectory "gerber/")
 		)
 	)
@@
 		(embedded_fonts no)
 	)
-	(footprint "Package_TO_SOT_THT:TO-92_Inline"
+	(footprint "Package_TO_SOT_THT:TO-92L_HandSolder"
 		(layer "F.Cu")
 		(at 133.23 101.36)
-		(descr "TO-92 leads in-line, narrow, oval pads, drill 0.75mm (see NXP sot054_po.pdf)")
+		(descr "TO-92L leads in-line (large body variant of TO-92), also known as TO-226, wide, drill 0.75mm, hand-soldering variant with enlarged pads (see https://www.diodes.com/assets/Package-Files/TO92L.pdf and http://www.ti.com/lit/an/snoa059/snoa059.pdf)")
 		(tags "to-92 sc-43 sc-43a sot54 PA33 transistor")
 		(property "Reference" "Q2"
-			(at 1.27 -3.56 0)
+			(at 1.27 -3.8 0)
 			(layer "F.SilkS")
 			(effects
@@
 			)
 		)
-		(property "Datasheet" "https://www.onsemi.com/pub/Collateral/BC550-D.pdf"
+		(property "Datasheet" ""
 			(at 0 0 0)
 			(unlocked yes)
@@
 			)
 		)
-		(property "Description" "0.1A Ic, 45V Vce, Small Signal NPN Transistor, TO-92"
+		(property "Description" ""
 			(at 0 0 0)
 			(unlocked yes)
@@
 		(sheetname "/")
 		(sheetfile "ember_launch_controller.kicad_sch")
-		(units
-			(unit
-				(name "A")
-				(pins "2" "1" "3")
-			)
-		)
 		(attr through_hole)
 		(duplicate_pad_numbers_are_jumpers no)
@@
 		)
 		(fp_arc
-			(start -0.568478 1.838478)
-			(mid -1.132087 -0.994977)
-			(end 1.27 -2.6)
+			(start -0.541453 1.842156)
+			(mid -1.247298 -0.581475)
+			(end 0.45 -2.45)
 			(stroke
 				(width 0.12)
@@
 		)
 		(fp_arc
-			(start 1.27 -2.6)
-			(mid 3.672087 -0.994977)
-			(end 3.108478 1.838478)
+			(start 2.05 -2.45)
+			(mid 3.769931 -0.601036)
+			(end 3.078445 1.827684)
 			(stroke
 				(width 0.12)
@@
 		)
 		(fp_line
-			(start -1.46 -2.73)
-			(end -1.46 2.01)
+			(start -1.46 -3.05)
+			(end 4 -3.05)
 			(stroke
 				(width 0.05)
@@
 		)
 		(fp_line
-			(start -1.46 -2.73)
-			(end 4 -2.73)
+			(start -1.45 -3.05)
+			(end -1.46 2.01)
 			(stroke
 				(width 0.05)
@@
 		(fp_line
 			(start 4 2.01)
-			(end 4 -2.73)
+			(end 4 -3.05)
 			(stroke
 				(width 0.05)
@@
 		)
 		(pad "1" thru_hole rect
-			(at 0 0)
-			(size 1.05 1.5)
-			(drill 0.75)
+			(at 0 0.25)
+			(size 1.4 2.1)
+			(drill 0.75
+				(offset 0 0.4)
+			)
 			(layers "*.Cu" "*.Mask")
 			(remove_unused_layers no)
@@
 			(pintype "passive")
 		)
-		(pad "2" thru_hole oval
-			(at 1.27 0)
-			(size 1.05 1.5)
-			(drill 0.75)
+		(pad "2" thru_hole roundrect
+			(at 1.27 -1.5)
+			(size 1.4 2.1)
+			(drill 0.75
+				(offset 0 -0.4)
+			)
 			(layers "*.Cu" "*.Mask")
 			(remove_unused_layers no)
+			(roundrect_rratio 0.25)
 			(net "Net-(Q2-B)")
 			(pinfunction "B_2")
 			(pintype "input")
 		)
-		(pad "3" thru_hole oval
-			(at 2.54 0)
-			(size 1.05 1.5)
-			(drill 0.75)
+		(pad "3" thru_hole roundrect
+			(at 2.54 0.25)
+			(size 1.4 2.1)
+			(drill 0.75
+				(offset 0 0.4)
+			)
 			(layers "*.Cu" "*.Mask")
 			(remove_unused_layers no)
+			(roundrect_rratio 0.25)
 			(net "GND")
 			(pinfunction "E_3")
@@
 		)
 		(embedded_fonts no)
-		(model "${KICAD10_3DMODEL_DIR}/Package_TO_SOT_THT.3dshapes/TO-92_Inline.step"
+		(model "${KICAD10_3DMODEL_DIR}/Package_TO_SOT_THT.3dshapes/TO-92L.step"
 			(offset
 				(xyz 0 0 0)
@@
 	)
 	(segment
-		(start 182 120.5)
-		(end 182 112.5)
+		(start 126.75 115.5)
+		(end 126.75 108.689942)
 		(width 0.4)
 		(layer "F.Cu")
@@
 	)
 	(segment
-		(start 131.685029 105.844971)
-		(end 129.594971 105.844971)
+		(start 182 120.5)
+		(end 182 112.5)
 		(width 0.4)
 		(layer "F.Cu")
@@
 	(segment
 		(start 127.75 116.5)
-		(end 131 116.5)
+		(end 126.75 115.5)
 		(width 0.4)
 		(layer "F.Cu")
@@
 	)
 	(segment
-		(start 126.75 115.5)
-		(end 127.75 116.5)
+		(start 135.77 102.83)
+		(end 135.77 101.61)
 		(width 0.4)
 		(layer "F.Cu")
@@
 	)
 	(segment
-		(start 129.594971 105.844971)
-		(end 126.75 108.689942)
+		(start 144 88.25)
+		(end 145.25 87)
 		(width 0.4)
 		(layer "F.Cu")
@@
 	)
 	(segment
-		(start 144 88.25)
-		(end 145.25 87)
+		(start 180.75 109.75)
+		(end 179 111.5)
 		(width 0.4)
 		(layer "F.Cu")
@@
 	)
 	(segment
-		(start 180.75 109.75)
-		(end 179 111.5)
+		(start 129.594971 105.844971)
+		(end 132.755029 105.844971)
 		(width 0.4)
 		(layer "F.Cu")
@@
 	)
 	(segment
+		(start 132.755029 105.844971)
+		(end 135.77 102.83)
+		(width 0.4)
+		(layer "F.Cu")
+		(net "GND")
+	)
+	(segment
 		(start 141.81 87)
 		(end 141.75 86.94)
@@
 	)
 	(segment
+		(start 126.75 108.689942)
+		(end 129.594971 105.844971)
+		(width 0.4)
+		(layer "F.Cu")
+		(net "GND")
+	)
+	(segment
 		(start 147 116.5)
 		(end 147 119.5)
@@
 	)
 	(segment
-		(start 135.77 101.76)
-		(end 131.685029 105.844971)
-		(width 0.4)
-		(layer "F.Cu")
-		(net "GND")
-	)
-	(segment
 		(start 148.5 87)
 		(end 145.25 87)
@@
 	)
 	(segment
-		(start 181.5 109.75)
-		(end 180.75 109.75)
+		(start 131 116.5)
+		(end 127.75 116.5)
 		(width 0.4)
 		(layer "F.Cu")
@@
 	)
 	(segment
-		(start 126.75 108.689942)
-		(end 126.75 115.5)
+		(start 181.5 109.75)
+		(end 180.75 109.75)
 		(width 0.4)
 		(layer "F.Cu")
@@
 	)
 	(segment
-		(start 141.75 94.56)
-		(end 135.06 94.56)
-		(width 0.4)
+		(start 134.5 100.09)
+		(end 134.5 95.12)
+		(width 0.2)
 		(layer "F.Cu")
 		(net "Net-(Q2-B)")
 	)
 	(segment
-		(start 134.5 99.76)
-		(end 134.5 95.12)
-		(width 0.4)
+		(start 134.5 95.12)
+		(end 135 94.62)
+		(width 0.2)
 		(layer "F.Cu")
 		(net "Net-(Q2-B)")
 	)
 	(segment
-		(start 135.06 94.56)
-		(end 135 94.62)
+		(start 141.75 94.56)
+		(end 135.06 94.56)
 		(width 0.4)
 		(layer "F.Cu")
@@
 	)
 	(segment
-		(start 134.5 95.12)
+		(start 135.06 94.56)
 		(end 135 94.62)
 		(width 0.4)
@@
 	)
 	(segment
-		(start 126 108.59)
-		(end 133.23 101.36)
-		(width 0.4)
-		(layer "F.Cu")
-		(net "Net-(BZ1--)")
-	)
-	(segment
 		(start 126 115.5)
 		(end 126 108.59)
@@
 	)
 	(segment
+		(start 126 108.59)
+		(end 133.23 101.36)
+		(width 0.4)
+		(layer "F.Cu")
+		(net "Net-(BZ1--)")
+	)
+	(segment
 		(start 139 109.5)
 		(end 139 102.25)
@@
 	)
 	(zone
+		(net "GND")
 		(layers "F.Cu" "B.Cu")
 		(name "1")
@@
 			(thermal_gap 0.5)
 			(thermal_bridge_width 0.5)
-			(island_removal_mode 1)
+			(island_removal_mode 0)
 		)
 		(polygon
@@
 			)
 		)
-	)
-	(zone
-		(net "GND")
-		(layers "F.Cu" "B.Cu")
-		(name "1")
-		(hatch edge 0.5)
-		(priority 1)
-		(connect_pads yes
-			(clearance 0.5)
-		)
-		(min_thickness 0.25)
-		(fill yes
-			(thermal_gap 0.5)
-			(thermal_bridge_width 0.5)
-			(island_removal_mode 1)
-		)
-		(polygon
-			(pts
-				(xy 175 100.5) (xy 174.899321 112.75) (xy 183.149321 112.75) (xy 183.25 100.5)
-			)
-		)
